Commit message: Experimental

File: models/materials.xacro (robot description, xacro)
@@ -8,5 +8,5 @@
     </material>
     <material name="white">
-        <color rgba="0.8 0.8 0.8 1"/>
+        <color rgba="0.8 0.8 0.8 0.5"/>
     </material>
     <material name="red">

File: models/myArm_brHand.xacro (robot description, xacro)
@@ -11,13 +11,18 @@
 <xacro:property name="PI"           value="3.1415926535897931"/>
 <xacro:property name="scale"        value="1" /> <!-- scale -->
-<xacro:property name="mass"         value="${1 * scale}"   /> <!-- arbitrary value for mass -->
-<xacro:property name="mass_divider" value="1"              /> <!-- mass divider -->
-<xacro:property name="radius"       value="${0.05 * scale}"/>
-<xacro:property name="radius2"      value="${0.5 * radius}"/>
-<xacro:property name="diameter"     value="${2 * radius}"  />
-<xacro:property name="baseLength"   value="${0.2 * scale}" /> <!-- base_link -->
-<xacro:property name="length1"      value="${0.5 * scale}" /> <!-- body 1 -->
-<xacro:property name="length10"     value="${4*radius}"    /> <!-- body 10 -->
-<xacro:property name="length2"      value="${0.5 * scale}" /> <!-- body 2 -->
+<xacro:property name="mass"         value="${1 * scale}"    /> <!-- arbitrary value for mass -->
+<xacro:property name="mass_divider" value="1"                /> <!-- mass divider -->
+<xacro:property name="radius_hor_2" value="${1 * radius2}" />
+<xacro:property name="radius_hor_3" value="${1 * radius3}" />
+<xacro:property name="baseLength"   value="${0.2 * scale}"   /> <!-- base_link -->
+<xacro:property name="base_radius"  value="${radius1}"       />
+<xacro:property name="length1"      value="${0.5 * scale}"   /> <!-- body 1 -->
+<xacro:property name="radius1"      value="${0.1 * scale}"   />
+<xacro:property name="length10"     value="${2*radius1}"     /> <!-- body 10 -->
+<xacro:property name="length2"      value="${0.5 * scale}"   /> <!-- body 2 -->
+<xacro:property name="radius2"      value="${0.1 * scale}"   />
+<xacro:property name="length20"     value="${2*radius1}"     /> <!-- body 20 -->
+<xacro:property name="length3"      value="${0.05 * scale}"  /> <!-- body 3 -->
+<xacro:property name="radius3"      value="${0.1 * scale}"  />
 <xacro:property name="damping"      value="1" />             <!-- Damping -->
 <xacro:property name="axel_offset"  value="0" />             <!-- Space btw top of beam and the each joint -->
@@ -39,5 +44,5 @@
         <origin xyz="0 0 0" rpy="0 0 0"/>
         <geometry>
-            <cylinder length="${baseLength}" radius="${radius}"/>
+            <cylinder length="${baseLength}" radius="${base_radius}"/>
         </geometry>
     </collision>
@@ -45,12 +50,14 @@
         <origin xyz="0 0 0" rpy="0 0 0"/>
         <geometry>
-            <cylinder length="${baseLength}" radius="${radius}"/>
+            <cylinder length="${baseLength}" radius="${base_radius}"/>
         </geometry>
         <material name ="white"/>
     </visual>
-    <inertial>  <!-- inertial -->
+    <!--
+    <inertial>  The root link base_link has an inertia specified in the URDF, but KDL does not support a root link with an inertia.  As a workaround, you can add an extra dummy link to your URDF.
         <origin xyz="0 0 0" rpy="0 0 0"/>
-        <xacro:cyl_inertia mass="${1/mass_divider}" h="${baseLength}" r="${radius}"/>
-    </inertial>
+        <xacro:cyl_inertia mass="${mass/mass_divider}" h="${baseLength}" r="${base_radius}"/>
+    </inertial>
+    -->
 </link>
 <!---............................. BASE JOINT REVOLUTE Z ................................-->
@@ -59,5 +66,5 @@
     <child link="body1"/>
     <axis xyz="0 0 1"/>
-    <origin rpy="0 0 0" xyz="0 0 0"/> <!-- z - offset (difference between two joint center) (Base link + Link1) length/2 -->
+    <origin rpy="0 0 0" xyz="0 0 ${baseLength/2+length1/2}"/> <!-- z - offset (difference between two joint center) (Base link + Link1) length/2 -->
     <limit effort="1000.0" lower="-2.96" upper="2.96" velocity="0.5"/>
     <dynamics damping="${damping}"/>
@@ -66,13 +73,13 @@
 <link name="body1">
     <collision> <!-- collision -->
-        <origin rpy="0 0 0" xyz="0 0 ${baseLength/2+length1/2}"/>
-        <geometry>
-            <cylinder length="${length1}" radius="${radius}"/>
+        <origin rpy="0 0 0" xyz="0 0 0"/>
+        <geometry>
+            <cylinder length="${length1}" radius="${radius1}"/>
         </geometry>
     </collision>
     <visual>    <!-- visual -->
-        <origin rpy="0 0 0" xyz="0 0 ${baseLength/2+length1/2}"/>
-        <geometry>
-            <cylinder length="${length1}" radius="${radius}"/>
+        <origin rpy="0 0 0" xyz="0 0 0"/>
+        <geometry>
+            <cylinder length="${length1}" radius="${radius1}"/>
         </geometry>
         <material name ="blue"/>
@@ -80,13 +87,14 @@
     <inertial>  <!-- inertial -->
         <origin rpy="0 0 0" xyz="0 0 0"/>
-        <xacro:cyl_inertia mass="${1/mass_divider}" h="${length1}" r="${radius}"/>
+        <xacro:cyl_inertia mass="${mass/mass_divider}" h="${length1}" r="${radius1}"/>
     </inertial>
 </link>
-<!---............................. JOINT 20 FIXED ................................-->
-<joint name="j20" type="fixed">
+<!---............................. JOINT 10 CONTINUOUS AROUND Y ................................-->
+<joint name="j10" type="continuous">
     <parent link="body1"/>
     <child link="body10"/>
-    <origin xyz="0 ${axel_offset} ${baseLength/2+length1+radius2}" rpy="0 0 0" />
-    <!-- <axis xyz="0 1 0"/> -->
+    <origin xyz="0 ${axel_offset} ${length1/2+radius_hor_2}" rpy="0 0 0" />
+    <axis xyz="0 1 0"/>
+    <limit effort="1000.0" lower="-2.96" upper="2.96" velocity="0.5"/>
     <dynamics damping="${damping}"/>
 </joint>
@@ -94,7 +102,7 @@
 <link name="body10">
     <collision> <!-- collision -->
-        <origin rpy="${PI/2} 0 0" xyz="0 0 0"/>
-        <geometry>
-            <cylinder length="${length10}" radius="${radius2}"/> <!-- Double the diameter of link cylinder-->
+        <origin rpy="${PI/2} 0 0" xyz="0 0 0"/> <!-- Due to being rotated around X, z as 0 -->
+        <geometry>
+            <cylinder length="${length10}" radius="${radius_hor_2}"/> <!-- Double the diameter of link cylinder-->
         </geometry>
     </collision>
@@ -102,5 +110,5 @@
         <origin rpy="${PI/2} 0 0" xyz="0 0 0"/>
         <geometry>
-            <cylinder length="${length10}" radius="${radius2}"/> <!-- Double the diameter of link cylinder-->
+            <cylinder length="${length10}" radius="${radius_hor_2}"/> <!-- Double the diameter of link cylinder-->
         </geometry>
         <material name ="white"/>
@@ -108,13 +116,13 @@
     <inertial>  <!-- inertial -->
         <origin rpy="0 0 0" xyz="0 0 0"/>
-        <xacro:cyl_inertia mass="${0.4/mass_divider}" h="${length10}" r="${radius2}"/>
+        <xacro:cyl_inertia mass="${mass/mass_divider}" h="${length10}" r="${radius_hor_2}"/>
     </inertial>
 </link>
-<!---............................. JOINT 2 REVOLUTE Y ................................-->
-<joint name="j2" type="revolute">
+<!---............................. JOINT 1 FIXED ................................-->
+<joint name="j1" type="fixed">
     <parent link="body10"/>
     <child link="body2"/>
     <origin xyz="0 ${axel_offset} 0" rpy="0 0 0"/>
-    <axis xyz="0 1 0"/>
+    <!-- <axis xyz="0 1 0"/> -->
     <limit effort="1000.0" lower="-2.96" upper="2.96" velocity="0.5"/>
     <dynamics damping="${damping}"/>
@@ -123,13 +131,13 @@
 <link name="body2">
     <collision> <!-- collision -->
-        <origin rpy="0 0 0" xyz="0 0 ${radius2+length2/2}"/>
-        <geometry>
-            <cylinder length="${length2}" radius="${radius}"/>
+        <origin rpy="0 0 0" xyz="0 0 ${radius_hor_2+length2/2}"/>
+        <geometry>
+            <cylinder length="${length2}" radius="${radius2}"/>
         </geometry>
     </collision>
     <visual>    <!-- visual -->
-        <origin rpy="0 0 0" xyz="0 0 ${radius2+length2/2}"/>
-        <geometry>
-            <cylinder length="${length2}" radius="${radius}"/>
+        <origin rpy="0 0 0" xyz="0 0 ${radius_hor_2+length2/2}"/>
+        <geometry>
+            <cylinder length="${length2}" radius="${radius2}"/>
         </geometry>
         <material name ="green"/>
@@ -137,15 +145,73 @@
     <inertial>  <!-- inertial -->
         <origin rpy="0 0 0" xyz="0 0 0"/>
-        <xacro:cyl_inertia mass="${1/mass_divider}" h="${length2}" r="${radius}"/>
+        <xacro:cyl_inertia mass="${mass/mass_divider}" h="${length2}" r="${radius2}"/>
     </inertial>
 </link>
-<!---............................. JOINT 3 REVOLUTE Y ................................-->
-<joint name="j3" type="revolute">
+<!---............................. JOINT 20 CONTINUOUS AROUND Y ................................-->
+<joint name="j20" type="continuous">
     <parent link="body2"/>
-    <child link="brHand"/>
-    <origin rpy="0 0 0" xyz="0 0 ${length2}"/>
+    <child link="body20"/>
+    <origin xyz="0 ${axel_offset} ${radius_hor_2 + length2 + radius_hor_3}" rpy="0 0 0" />
     <axis xyz="0 1 0"/>
     <limit effort="1000.0" lower="-2.96" upper="2.96" velocity="0.5"/>
     <dynamics damping="${damping}"/>
+</joint>
+<!---............................. LINK 20 WHITE ................................-->
+<link name="body20">
+    <collision> <!-- collision -->
+        <origin rpy="${PI/2} 0 0" xyz="0 0 0"/>
+        <geometry>
+            <cylinder length="${length20}" radius="${radius_hor_3}"/> <!-- Double the diameter of link cylinder-->
+        </geometry>
+    </collision>
+    <visual>    <!-- visual -->
+        <origin rpy="${PI/2} 0 0" xyz="0 0 0"/>
+        <geometry>
+            <cylinder length="${length20}" radius="${radius_hor_3}"/> <!-- Double the diameter of link cylinder-->
+        </geometry>
+        <material name ="white"/>
+    </visual>
+    <inertial>  <!-- inertial -->
+        <origin rpy="0 0 0" xyz="0 0 0"/>
+        <xacro:cyl_inertia mass="${mass/mass_divider}" h="${length20}" r="${radius_hor_3}"/>
+    </inertial>
+</link>
+<!---............................. JOINT 2 FIXED ................................-->
+<joint name="j2" type="fixed">
+    <parent link="body20"/>
+    <child link="body3"/>
+    <origin xyz="0 ${axel_offset} 0" rpy="0 0 0"/>
+    <!--<axis xyz="0 1 0"/> -->
+    <limit effort="1000.0" lower="-2.96" upper="2.96" velocity="0.5"/>
+    <dynamics damping="${damping}"/>
+</joint>
+<!---............................. LINK 3 GREEN .......................................-->
+<link name="body3">
+    <collision> <!-- collision -->
+        <origin rpy="0 0 0" xyz="0 0 ${radius_hor_3+length3/2}"/>
+        <geometry>
+            <cylinder length="${length3}" radius="${radius3}"/>
+        </geometry>
+    </collision>
+    <visual>    <!-- visual -->
+        <origin rpy="0 0 0" xyz="0 0 ${radius_hor_3+length3/2}"/>
+        <geometry>
+            <cylinder length="${length3}" radius="${radius3}"/>
+        </geometry>
+        <material name ="green"/>
+    </visual>
+    <inertial>  <!-- inertial -->
+        <origin rpy="0 0 0" xyz="0 0 0"/>
+        <xacro:cyl_inertia mass="${mass/mass_divider}" h="${length3}" r="${radius3}"/>
+    </inertial>
+</link>
+<!---............................. JOINT 3 REVOLUTE Z ................................-->
+<joint name="j3" type="revolute">
+    <parent link="body3"/>
+    <child link="brHand"/>
+    <origin xyz="0 ${axel_offset} ${radius_hor_3+length3}" rpy="0 0 0"/>
+    <axis xyz="0 0 1"/>
+    <limit effort="1000.0" lower="-2.96" upper="2.96" velocity="0.5"/>
+    <dynamics damping="${2 * damping}"/>
 </joint>
 <!---............................. HAND .............................................. -->
@@ -189,54 +255,13 @@
     </collision>
   </link>
-  <link
-    name="finger_1_prox_link">
-    <inertial>
-      <origin
-        xyz="-0.0288648917008988 9.98379746692153E-05 0.0171253477569802"
-        rpy="0 0 0" />
-      <mass
-        value="56143.0626955765" />
-      <inertia
-        ixx="10.4484040652085"
-        ixy="-0.117861448219975"
-        ixz="-5.31613760585343"
-        iyy="33.9552353012776"
-        iyz="0.0780041192837706"
-        izz="29.3669090518615" />
-    </inertial>
-    <visual>
-      <origin
-        xyz="0 0 0"
-        rpy="0 0 0" />
-      <geometry>
-        <mesh
-          filename="package://my_arm/meshes/finger_1_prox_link.STL" scale="1.5 1.5 1.5"/>
-      </geometry>
-      <material
-        name="">
-        <color
-          rgba="0.752941176470588 0.752941176470588 0.752941176470588 1" />
-      </material>
-    </visual>
-    <collision>
-      <origin
-        xyz="0 0 0"
-        rpy="0 0 0" />
-      <geometry>
-        <mesh
-          filename="package://my_arm/meshes/finger_1_prox_link.STL" scale="1.5 1.5 1.5"/>
-      </geometry>
-    </collision>
-  </link>
   <joint
-    name="finger_1_prox_joint"
-    type="revolute">
-    <origin
-      xyz="0.025 0 0.0415"
-      rpy="0 2.7051E-17 -1.5708" />
+    name="finger_1_prox_joint" type="revolute">
     <parent
       link="brHand" />
     <child
       link="finger_1_prox_link" />
+    <origin
+      xyz="0.025 0 0.0415"
+      rpy="0 2.7051E-17 -1.5708" />
     <axis
       xyz="0 0 1" />
@@ -248,4 +273,44 @@
     <dynamics damping="${damping}"/>
   </joint>
+  <link
+    name="finger_1_prox_link">
+    <inertial>
+      <origin
+        xyz="-0.0288648917008988 9.98379746692153E-05 0.0171253477569802"
+        rpy="0 0 0" />
+      <mass
+        value="56143.0626955765" />
+      <inertia
+        ixx="10.4484040652085"
+        ixy="-0.117861448219975"
+        ixz="-5.31613760585343"
+        iyy="33.9552353012776"
+        iyz="0.0780041192837706"
+        izz="29.3669090518615" />
+    </inertial>
+    <visual>
+      <origin
+        xyz="0 0 0"
+        rpy="0 0 0" />
+      <geometry>
+        <mesh
+          filename="package://my_arm/meshes/finger_1_prox_link.STL" scale="1.5 1.5 1.5"/>
+      </geometry>
+      <material
+        name="">
+        <color
+          rgba="0.752941176470588 0.752941176470588 0.752941176470588 1" />
+      </material>
+    </visual>
+    <collision>
+      <origin
+        xyz="0 0 0"
+        rpy="0 0 0" />
+      <geometry>
+        <mesh
+          filename="package://my_arm/meshes/finger_1_prox_link.STL" scale="1.5 1.5 1.5"/>
+      </geometry>
+    </collision>
+  </link>
   <link
     name="finger_1_med_liink">
