Commit message: Add Jaco Arm model.

File: models/myArm_brHand.xacro (robot description, xacro)
@@ -1,13 +1,25 @@
 <?xml version="1.0"?>
 <robot name="robotArm" xmlns:xacro="http://www.ros.org/wiki/xacro">
+<!-- Formula according to https://en.wikipedia.org/wiki/List_of_moment_of_inertia_tensors for cylinder -->
+<xacro:macro name="cyl_inertia" params="mass r h ">
+    <mass value="${mass}"/>
+    <inertia ixx="${0.083333 * mass * (3*r*r + h*h)}" ixy="0" ixz="0"
+             iyy="${0.083333 * mass * (3*r*r + h*h)}" iyz="0"
+             izz="${0.5*mass*r*r}" />
+</xacro:macro>
 <!-- Constants for robot dimensions -->
-<xacro:property name="PI" value="3.1415926535897931"/>
-<xacro:property name="mass" value="1" /> <!-- arbitrary value for mass -->
-<xacro:property name="radius" value="0.2" />
-<xacro:property name="baseLength" value="0.2" /> <!-- base_link -->
-<xacro:property name="length1"  value="1" />     <!-- body 1 -->
-<xacro:property name="length10" value="0.8" />   <!-- body 10 -->
-<xacro:property name="length2"  value="1" />     <!-- body 2 -->
-<xacro:property name="axel_offset" value="0.05" /> <!-- Space btw top of beam and the each joint -->
+<xacro:property name="PI"           value="3.1415926535897931"/>
+<xacro:property name="scale"        value="1" /> <!-- scale -->
+<xacro:property name="mass"         value="${1 * scale}"   /> <!-- arbitrary value for mass -->
+<xacro:property name="mass_divider" value="1"              /> <!-- mass divider -->
+<xacro:property name="radius"       value="${0.05 * scale}"/>
+<xacro:property name="radius2"      value="${0.5 * radius}"/>
+<xacro:property name="diameter"     value="${2 * radius}"  />
+<xacro:property name="baseLength"   value="${0.2 * scale}" /> <!-- base_link -->
+<xacro:property name="length1"      value="${0.5 * scale}" /> <!-- body 1 -->
+<xacro:property name="length10"     value="${4*radius}"    /> <!-- body 10 -->
+<xacro:property name="length2"      value="${0.5 * scale}" /> <!-- body 2 -->
+<xacro:property name="damping"      value="1" />             <!-- Damping -->
+<xacro:property name="axel_offset"  value="0" />             <!-- Space btw top of beam and the each joint -->
 <!-- Import all Gazebo-customization elements, including Gazebo colors -->
 <xacro:include filename="$(find my_arm)/models/myArm2.gazebo" />
@@ -15,13 +27,15 @@
 <xacro:include filename="$(find my_arm)/models/materials.xacro" />
 <!---............................. Link Definitions ................................-->
-<link name="world"/>
-<joint name="fixed" type="fixed">
-  <parent link="world"/>
-  <child link="base_link"/>
+<!--
+<link name="root"/>
+<joint name="root_joint" type="fixed">
+    <parent link="root"/>
+    <child link="base_link"/>
 </joint>
-<!---............................. BASE LINK RED ................................-->
+-->
+<!---............................. BASE LINK WHITE ................................-->
 <link name="base_link">
     <collision> <!-- collision -->
-        <origin xyz="0 0 ${baseLength/2}" rpy="0 0 0"/>
+        <origin xyz="0 0 0" rpy="0 0 0"/>
         <geometry>
             <cylinder length="${baseLength}" radius="${radius}"/>
@@ -29,5 +43,5 @@
     </collision>
     <visual>    <!-- visual -->
-        <origin xyz="0 0 ${baseLength/2}" rpy="0 0 0"/>
+        <origin xyz="0 0 0" rpy="0 0 0"/>
         <geometry>
             <cylinder length="${baseLength}" radius="${radius}"/>
@@ -36,10 +50,6 @@
     </visual>
     <inertial>  <!-- inertial -->
-        <origin xyz="0 0 ${baseLength/2}" rpy="0 0 0"/>
-        <mass value="${mass}"/>
-        <inertia
-            ixx="${mass / 12.0 * (2*PI*radius*baseLength)}" ixy="0.0" ixz="0.0"
-            iyy="${mass / 12.0 * (2*PI*radius*baseLength)}" iyz="0.0"
-            izz="${mass / 12.0 * (2*PI*radius*radius)}"/>
+        <origin xyz="0 0 0" rpy="0 0 0"/>
+        <xacro:cyl_inertia mass="${1/mass_divider}" h="${baseLength}" r="${radius}"/>
     </inertial>
 </link>
@@ -49,29 +59,26 @@
     <child link="body1"/>
     <axis xyz="0 0 1"/>
-    <origin rpy="0 0 0" xyz="0 0 0.6"/> <!-- z - offset (difference between two joint center) (Base link + Link1) length/2 -->
+    <origin rpy="0 0 0" xyz="0 0 0"/> <!-- z - offset (difference between two joint center) (Base link + Link1) length/2 -->
     <limit effort="1000.0" lower="-2.96" upper="2.96" velocity="0.5"/>
+    <dynamics damping="${damping}"/>
 </joint>
-<!---............................. LINK 1 YELLOW ................................-->
+<!---............................. LINK 1 BLUE ................................-->
 <link name="body1">
     <collision> <!-- collision -->
+        <origin rpy="0 0 0" xyz="0 0 ${baseLength/2+length1/2}"/>
+        <geometry>
+            <cylinder length="${length1}" radius="${radius}"/>
+        </geometry>
+    </collision>
+    <visual>    <!-- visual -->
+        <origin rpy="0 0 0" xyz="0 0 ${baseLength/2+length1/2}"/>
+        <geometry>
+            <cylinder length="${length1}" radius="${radius}"/>
+        </geometry>
+        <material name ="blue"/>
+    </visual>
+    <inertial>  <!-- inertial -->
         <origin rpy="0 0 0" xyz="0 0 0"/>
-        <geometry>
-            <cylinder length="${length1}" radius="${radius}"/>
-        </geometry>
-    </collision>
-    <visual>    <!-- visual -->
-        <origin rpy="0 0 0" xyz="0 0 0"/>
-        <geometry>
-            <cylinder length="${length1}" radius="${radius}"/>
-        </geometry>
-        <material name ="blue"/>
-    </visual>
-    <inertial>  <!-- inertial -->
-        <origin xyz="0 0 ${length1/2 - axel_offset}" rpy="0 0 0"/>
-        <mass value="${mass}"/>
-        <inertia
-            ixx="${mass / 12.0 * (2*PI*radius*length1)}" ixy="0.0" ixz="0.0"
-            iyy="${mass / 12.0 * (2*PI*radius*length1)}" iyz="0.0"
-            izz="${mass / 12.0 * (2*PI*radius*radius)}"/>
+        <xacro:cyl_inertia mass="${1/mass_divider}" h="${length1}" r="${radius}"/>
     </inertial>
 </link>
@@ -80,30 +87,26 @@
     <parent link="body1"/>
     <child link="body10"/>
-    <axis xyz="1 0 0"/>
-    <origin rpy="0 0 0" xyz="0 0.2 0.7"/>
-    <limit effort="1000.0" lower="-2.96" upper="2.96" velocity="0.5"/>
+    <origin xyz="0 ${axel_offset} ${baseLength/2+length1+radius2}" rpy="0 0 0" />
+    <!-- <axis xyz="0 1 0"/> -->
+    <dynamics damping="${damping}"/>
 </joint>
-<!---............................. LINK 10 DUMP WHITE ................................-->
+<!---............................. LINK 10 WHITE ................................-->
 <link name="body10">
     <collision> <!-- collision -->
-        <origin rpy="1.57 0 0" xyz="0 0 0"/>
-        <geometry>
-            <cylinder length="${length10}" radius="${radius}"/> <!-- Double the diameter of link cylinder-->
+        <origin rpy="${PI/2} 0 0" xyz="0 0 0"/>
+        <geometry>
+            <cylinder length="${length10}" radius="${radius2}"/> <!-- Double the diameter of link cylinder-->
         </geometry>
     </collision>
     <visual>    <!-- visual -->
-        <origin rpy="1.57 0 0" xyz="0 0 0"/>
-        <geometry>
-            <cylinder length="${length10}" radius="${radius}"/> <!-- Double the diameter of link cylinder-->
+        <origin rpy="${PI/2} 0 0" xyz="0 0 0"/>
+        <geometry>
+            <cylinder length="${length10}" radius="${radius2}"/> <!-- Double the diameter of link cylinder-->
         </geometry>
         <material name ="white"/>
     </visual>
     <inertial>  <!-- inertial -->
-        <origin xyz="0 0 ${length10/2 - axel_offset}" rpy="0 0 0"/>
-        <mass value="${mass}"/>
-        <inertia
-            ixx="${mass / 12.0 * (2*PI*radius*length10)}" ixy="0.0" ixz="0.0"
-            iyy="${mass / 12.0 * (2*PI*radius*length10)}" iyz="0.0"
-            izz="${mass / 12.0 * (2*PI*radius*radius)}"/>
+        <origin rpy="0 0 0" xyz="0 0 0"/>
+        <xacro:cyl_inertia mass="${0.4/mass_divider}" h="${length10}" r="${radius2}"/>
     </inertial>
 </link>
@@ -112,30 +115,27 @@
     <parent link="body10"/>
     <child link="body2"/>
+    <origin xyz="0 ${axel_offset} 0" rpy="0 0 0"/>
     <axis xyz="0 1 0"/>
-    <origin rpy="0 0 0" xyz="0 0.2 0.3"/>
     <limit effort="1000.0" lower="-2.96" upper="2.96" velocity="0.5"/>
+    <dynamics damping="${damping}"/>
 </joint>
 <!---............................. LINK 2 GREEN .......................................-->
 <link name="body2">
     <collision> <!-- collision -->
+        <origin rpy="0 0 0" xyz="0 0 ${radius2+length2/2}"/>
+        <geometry>
+            <cylinder length="${length2}" radius="${radius}"/>
+        </geometry>
+    </collision>
+    <visual>    <!-- visual -->
+        <origin rpy="0 0 0" xyz="0 0 ${radius2+length2/2}"/>
+        <geometry>
+            <cylinder length="${length2}" radius="${radius}"/>
+        </geometry>
+        <material name ="green"/>
+    </visual>
+    <inertial>  <!-- inertial -->
         <origin rpy="0 0 0" xyz="0 0 0"/>
-        <geometry>
-            <cylinder length="${length2}" radius="${radius}"/>
-        </geometry>
-    </collision>
-    <visual>    <!-- visual -->
-        <origin rpy="0 0 0" xyz="0 0 0"/>
-        <geometry>
-            <cylinder length="${length2}" radius="${radius}"/>
-        </geometry>
-        <material name ="green"/>
-    </visual>
-    <inertial>  <!-- inertial -->
-        <origin xyz="0 0 ${length2/2 - axel_offset}" rpy="0 0 0"/>
-        <mass value="${mass}"/>
-        <inertia
-            ixx="${mass / 12.0 * (2*PI*radius*length2)}" ixy="0.0" ixz="0.0"
-            iyy="${mass / 12.0 * (2*PI*radius*length2)}" iyz="0.0"
-            izz="${mass / 12.0 * (2*PI*radius*radius)}"/>
+        <xacro:cyl_inertia mass="${1/mass_divider}" h="${length2}" r="${radius}"/>
     </inertial>
 </link>
@@ -144,9 +144,10 @@
     <parent link="body2"/>
     <child link="brHand"/>
-    <origin rpy="0 0 0" xyz="0 0 0.6"/>
+    <origin rpy="0 0 0" xyz="0 0 ${length2}"/>
     <axis xyz="0 1 0"/>
     <limit effort="1000.0" lower="-2.96" upper="2.96" velocity="0.5"/>
+    <dynamics damping="${damping}"/>
 </joint>
-<!---............................. HAND ..............................................-->
+<!---............................. HAND .............................................. -->
   <link name="brHand">
     <inertial>
@@ -245,4 +246,5 @@
       effort="0"
       velocity="0" />
+    <dynamics damping="${damping}"/>
   </joint>
   <link
@@ -303,4 +305,5 @@
       effort="0"
       velocity="0" />
+    <dynamics damping="${damping}"/>
   </joint>
   <link
@@ -361,4 +364,5 @@
       effort="0"
       velocity="0" />
+    <dynamics damping="${damping}"/>
   </joint>
   <link
@@ -419,4 +423,5 @@
       effort="0"
       velocity="0" />
+    <dynamics damping="${damping}"/>
   </joint>
   <link
@@ -477,4 +482,5 @@
       effort="0"
       velocity="0" />
+    <dynamics damping="${damping}"/>
   </joint>
   <link
@@ -535,4 +541,5 @@
       effort="0"
       velocity="0" />
+    <dynamics damping="${damping}"/>
   </joint>
   <link
@@ -593,4 +600,5 @@
       effort="0"
       velocity="0" />
+    <dynamics damping="${damping}"/>
   </joint>
   <link
@@ -651,4 +659,5 @@
       effort="0"
       velocity="0" />
+    <dynamics damping="${damping}"/>
   </joint>
 </robot>

Commit message: Add Interactive Markers

File: models/myArm_brHand.xacro (robot description, xacro)
@@ -90,6 +90,6 @@
     </inertial>
 </link>
-<!---............................. JOINT 10 CONTINUOUS AROUND Y ................................-->
-<joint name="j10" type="continuous">
+<!---............................. JOINT 1 CONTINUOUS AROUND Y ................................-->
+<joint name="j1" type="continuous">
     <parent link="body1"/>
     <child link="body10"/>
@@ -120,5 +120,5 @@
 </link>
 <!---............................. JOINT 1 FIXED ................................-->
-<joint name="j1" type="fixed">
+<joint name="j10" type="fixed">
     <parent link="body10"/>
     <child link="body2"/>
@@ -149,5 +149,5 @@
 </link>
 <!---............................. JOINT 20 CONTINUOUS AROUND Y ................................-->
-<joint name="j20" type="continuous">
+<joint name="j2" type="continuous">
     <parent link="body2"/>
     <child link="body20"/>
@@ -178,5 +178,5 @@
 </link>
 <!---............................. JOINT 2 FIXED ................................-->
-<joint name="j2" type="fixed">
+<joint name="j20" type="fixed">
     <parent link="body20"/>
     <child link="body3"/>
