Commit message: Improve theta2 calculation Add PISA-IIT SoftHand

File: models/myArm_brHand.urdf (robot description, URDF)
Before this commit: robot robotArm, 13 links, 12 joints
Links:
- removed link body1
- removed link body10
- added link body20; visual cylinder length=0.8 radius=0.2
- added link body3; visual cylinder length=1 radius=0.2
Joints:
- removed joint j2
- removed joint j20
- added joint j30: type fixed, parent body2, child body20, origin xyz=0 0.2 0.7 rpy=0 0 0, axis 1 0 0, limit lower=-2.96 upper=2.96 effort=1000.0 velocity=0.5
- added joint j4: type revolute, parent body3, child brHand, origin xyz=0 0 0.6 rpy=0 0 0, axis 0 1 0, limit lower=-2.96 upper=2.96 effort=1000.0 velocity=0.5
- joint base_joint: child body1 -> body2
- joint j3: child brHand -> body3; origin xyz=0 0 0.6 rpy=0 0 0 -> xyz=0 0.2 0.3 rpy=0 0 0; parent body2 -> body20

File: models/myArm_brHand.xacro (robot description, xacro)
@@ -13,16 +13,16 @@
 <xacro:property name="mass"         value="${1 * scale}"    /> <!-- arbitrary value for mass -->
 <xacro:property name="mass_divider" value="1"                /> <!-- mass divider -->
-<xacro:property name="radius_hor_2" value="${1 * radius2}" />
-<xacro:property name="radius_hor_3" value="${1 * radius3}" />
+<xacro:property name="radius_hor_2" value="${1 * radius3}" />
+<xacro:property name="radius_hor_3" value="${1 * radius4}" />
 <xacro:property name="baseLength"   value="${0.2 * scale}"   /> <!-- base_link -->
-<xacro:property name="base_radius"  value="${radius1}"       />
-<xacro:property name="length1"      value="${0.5 * scale}"   /> <!-- body 1 -->
-<xacro:property name="radius1"      value="${0.1 * scale}"   />
-<xacro:property name="length10"     value="${2*radius1}"     /> <!-- body 10 -->
+<xacro:property name="base_radius"  value="${radius2}"       />
 <xacro:property name="length2"      value="${0.5 * scale}"   /> <!-- body 2 -->
 <xacro:property name="radius2"      value="${0.1 * scale}"   />
-<xacro:property name="length20"     value="${2*radius1}"     /> <!-- body 20 -->
-<xacro:property name="length3"      value="${0.05 * scale}"  /> <!-- body 3 -->
-<xacro:property name="radius3"      value="${0.1 * scale}"  />
+<xacro:property name="length20"     value="${2*radius2}"     /> <!-- body 20 -->
+<xacro:property name="length3"      value="${0.5 * scale}"   /> <!-- body 3 -->
+<xacro:property name="radius3"      value="${0.1 * scale}"   />
+<xacro:property name="length30"     value="${2*radius2}"     /> <!-- body 30 -->
+<xacro:property name="length4"      value="${0.3 * scale}"   /> <!-- body 4 -->
+<xacro:property name="radius4"      value="${0.1 * scale}"  />
 <xacro:property name="damping"      value="1" />             <!-- Damping -->
 <xacro:property name="axel_offset"  value="0" />             <!-- Space btw top of beam and the each joint -->
@@ -64,16 +64,16 @@
 <joint name="base_joint" type="revolute">
     <parent link="base_link"/>
-    <child link="body1"/>
+    <child link="body2"/>
     <axis xyz="0 0 1"/>
-    <origin rpy="0 0 0" xyz="0 0 ${baseLength/2+length1/2}"/> <!-- z - offset (difference between two joint center) (Base link + Link1) length/2 -->
+    <origin rpy="0 0 0" xyz="0 0 ${baseLength/2+length2/2}"/> <!-- z - offset (difference between two joint center) (Base link + Link1) length/2 -->
     <limit effort="1000.0" lower="-2.96" upper="2.96" velocity="0.5"/>
     <dynamics damping="${damping}"/>
 </joint>
-<!---............................. LINK 1 BLUE ................................-->
-<link name="body1">
+<!---............................. LINK 2 BLUE ................................-->
+<link name="body2">
     <collision> <!-- collision -->
         <origin rpy="0 0 0" xyz="0 0 0"/>
         <geometry>
-            <cylinder length="${length1}" radius="${radius1}"/>
+            <cylinder length="${length2}" radius="${radius2}"/>
         </geometry>
     </collision>
@@ -81,65 +81,7 @@
         <origin rpy="0 0 0" xyz="0 0 0"/>
         <geometry>
-            <cylinder length="${length1}" radius="${radius1}"/>
+            <cylinder length="${length2}" radius="${radius2}"/>
         </geometry>
         <material name ="blue"/>
-    </visual>
-    <inertial>  <!-- inertial -->
-        <origin rpy="0 0 0" xyz="0 0 0"/>
-        <xacro:cyl_inertia mass="${mass/mass_divider}" h="${length1}" r="${radius1}"/>
-    </inertial>
-</link>
-<!---............................. JOINT 1 CONTINUOUS AROUND Y ................................-->
-<joint name="j1" type="continuous">
-    <parent link="body1"/>
-    <child link="body10"/>
-    <origin xyz="0 ${axel_offset} ${length1/2+radius_hor_2}" rpy="0 0 0" />
-    <axis xyz="0 1 0"/>
-    <limit effort="1000.0" lower="-2.96" upper="2.96" velocity="0.5"/>
-    <dynamics damping="${damping}"/>
-</joint>
-<!---............................. LINK 10 WHITE ................................-->
-<link name="body10">
-    <collision> <!-- collision -->
-        <origin rpy="${PI/2} 0 0" xyz="0 0 0"/> <!-- Due to being rotated around X, z as 0 -->
-        <geometry>
-            <cylinder length="${length10}" radius="${radius_hor_2}"/> <!-- Double the diameter of link cylinder-->
-        </geometry>
-    </collision>
-    <visual>    <!-- visual -->
-        <origin rpy="${PI/2} 0 0" xyz="0 0 0"/>
-        <geometry>
-            <cylinder length="${length10}" radius="${radius_hor_2}"/> <!-- Double the diameter of link cylinder-->
-        </geometry>
-        <material name ="white"/>
-    </visual>
-    <inertial>  <!-- inertial -->
-        <origin rpy="0 0 0" xyz="0 0 0"/>
-        <xacro:cyl_inertia mass="${mass/mass_divider}" h="${length10}" r="${radius_hor_2}"/>
-    </inertial>
-</link>
-<!---............................. JOINT 1 FIXED ................................-->
-<joint name="j10" type="fixed">
-    <parent link="body10"/>
-    <child link="body2"/>
-    <origin xyz="0 ${axel_offset} 0" rpy="0 0 0"/>
-    <!-- <axis xyz="0 1 0"/> -->
-    <limit effort="1000.0" lower="-2.96" upper="2.96" velocity="0.5"/>
-    <dynamics damping="${damping}"/>
-</joint>
-<!---............................. LINK 2 GREEN .......................................-->
-<link name="body2">
-    <collision> <!-- collision -->
-        <origin rpy="0 0 0" xyz="0 0 ${radius_hor_2+length2/2}"/>
-        <geometry>
-            <cylinder length="${length2}" radius="${radius2}"/>
-        </geometry>
-    </collision>
-    <visual>    <!-- visual -->
-        <origin rpy="0 0 0" xyz="0 0 ${radius_hor_2+length2/2}"/>
-        <geometry>
-            <cylinder length="${length2}" radius="${radius2}"/>
-        </geometry>
-        <material name ="green"/>
     </visual>
     <inertial>  <!-- inertial -->
@@ -148,9 +90,9 @@
     </inertial>
 </link>
-<!---............................. JOINT 20 CONTINUOUS AROUND Y ................................-->
+<!---............................. JOINT 2 CONTINUOUS AROUND Y ................................-->
 <joint name="j2" type="continuous">
     <parent link="body2"/>
     <child link="body20"/>
-    <origin xyz="0 ${axel_offset} ${radius_hor_2 + length2 + radius_hor_3}" rpy="0 0 0" />
+    <origin xyz="0 ${axel_offset} ${length2/2+radius_hor_2}" rpy="0 0 0" />
     <axis xyz="0 1 0"/>
     <limit effort="1000.0" lower="-2.96" upper="2.96" velocity="0.5"/>
@@ -160,7 +102,7 @@
 <link name="body20">
     <collision> <!-- collision -->
-        <origin rpy="${PI/2} 0 0" xyz="0 0 0"/>
-        <geometry>
-            <cylinder length="${length20}" radius="${radius_hor_3}"/> <!-- Double the diameter of link cylinder-->
+        <origin rpy="${PI/2} 0 0" xyz="0 0 0"/> <!-- Due to being rotated around X, z as 0 -->
+        <geometry>
+            <cylinder length="${length20}" radius="${radius_hor_2}"/> <!-- Double the diameter of link cylinder-->
         </geometry>
     </collision>
@@ -168,5 +110,5 @@
         <origin rpy="${PI/2} 0 0" xyz="0 0 0"/>
         <geometry>
-            <cylinder length="${length20}" radius="${radius_hor_3}"/> <!-- Double the diameter of link cylinder-->
+            <cylinder length="${length20}" radius="${radius_hor_2}"/> <!-- Double the diameter of link cylinder-->
         </geometry>
         <material name ="white"/>
@@ -174,5 +116,5 @@
     <inertial>  <!-- inertial -->
         <origin rpy="0 0 0" xyz="0 0 0"/>
-        <xacro:cyl_inertia mass="${mass/mass_divider}" h="${length20}" r="${radius_hor_3}"/>
+        <xacro:cyl_inertia mass="${mass/mass_divider}" h="${length20}" r="${radius_hor_2}"/>
     </inertial>
 </link>
@@ -182,5 +124,5 @@
     <child link="body3"/>
     <origin xyz="0 ${axel_offset} 0" rpy="0 0 0"/>
-    <!--<axis xyz="0 1 0"/> -->
+    <!-- <axis xyz="0 1 0"/> -->
     <limit effort="1000.0" lower="-2.96" upper="2.96" velocity="0.5"/>
     <dynamics damping="${damping}"/>
@@ -189,5 +131,5 @@
 <link name="body3">
     <collision> <!-- collision -->
-        <origin rpy="0 0 0" xyz="0 0 ${radius_hor_3+length3/2}"/>
+        <origin rpy="0 0 0" xyz="0 0 ${radius_hor_2+length3/2}"/>
         <geometry>
             <cylinder length="${length3}" radius="${radius3}"/>
@@ -195,5 +137,5 @@
     </collision>
     <visual>    <!-- visual -->
-        <origin rpy="0 0 0" xyz="0 0 ${radius_hor_3+length3/2}"/>
+        <origin rpy="0 0 0" xyz="0 0 ${radius_hor_2+length3/2}"/>
         <geometry>
             <cylinder length="${length3}" radius="${radius3}"/>
@@ -206,9 +148,67 @@
     </inertial>
 </link>
-<!---............................. JOINT 3 REVOLUTE Z ................................-->
-<joint name="j3" type="revolute">
+<!---............................. JOINT 20 CONTINUOUS AROUND Y ................................-->
+<joint name="j3" type="continuous">
     <parent link="body3"/>
+    <child link="body30"/>
+    <origin xyz="0 ${axel_offset} ${radius_hor_2 + length3 + radius_hor_3}" rpy="0 0 0" />
+    <axis xyz="0 1 0"/>
+    <limit effort="1000.0" lower="-2.96" upper="2.96" velocity="0.5"/>
+    <dynamics damping="${damping}"/>
+</joint>
+<!---............................. LINK 30 WHITE ................................-->
+<link name="body30">
+    <collision> <!-- collision -->
+        <origin rpy="${PI/2} 0 0" xyz="0 0 0"/>
+        <geometry>
+            <cylinder length="${length30}" radius="${radius_hor_3}"/> <!-- Double the diameter of link cylinder-->
+        </geometry>
+    </collision>
+    <visual>    <!-- visual -->
+        <origin rpy="${PI/2} 0 0" xyz="0 0 0"/>
+        <geometry>
+            <cylinder length="${length30}" radius="${radius_hor_3}"/> <!-- Double the diameter of link cylinder-->
+        </geometry>
+        <material name ="white"/>
+    </visual>
+    <inertial>  <!-- inertial -->
+        <origin rpy="0 0 0" xyz="0 0 0"/>
+        <xacro:cyl_inertia mass="${mass/mass_divider}" h="${length30}" r="${radius_hor_3}"/>
+    </inertial>
+</link>
+<!---............................. JOINT 3 FIXED ................................-->
+<joint name="j30" type="fixed">
+    <parent link="body30"/>
+    <child link="body4"/>
+    <origin xyz="0 ${axel_offset} 0" rpy="0 0 0"/>
+    <!--<axis xyz="0 1 0"/> -->
+    <limit effort="1000.0" lower="-2.96" upper="2.96" velocity="0.5"/>
+    <dynamics damping="${damping}"/>
+</joint>
+<!---............................. LINK 4 GREEN .......................................-->
+<link name="body4">
+    <collision> <!-- collision -->
+        <origin rpy="0 0 0" xyz="0 0 ${radius_hor_3+length4/2}"/>
+        <geometry>
+            <cylinder length="${length4}" radius="${radius4}"/>
+        </geometry>
+    </collision>
+    <visual>    <!-- visual -->
+        <origin rpy="0 0 0" xyz="0 0 ${radius_hor_3+length4/2}"/>
+        <geometry>
+            <cylinder length="${length4}" radius="${radius4}"/>
+        </geometry>
+        <material name ="green"/>
+    </visual>
+    <inertial>  <!-- inertial -->
+        <origin rpy="0 0 0" xyz="0 0 0"/>
+        <xacro:cyl_inertia mass="${mass/mass_divider}" h="${length4}" r="${radius4}"/>
+    </inertial>
+</link>
+<!---............................. JOINT 4 REVOLUTE Z ................................-->
+<joint name="j4" type="revolute">
+    <parent link="body4"/>
     <child link="brHand"/>
-    <origin xyz="0 ${axel_offset} ${radius_hor_3+length3}" rpy="0 0 0"/>
+    <origin xyz="0 ${axel_offset} ${radius_hor_3+length4}" rpy="0 0 0"/>
     <axis xyz="0 0 1"/>
     <limit effort="1000.0" lower="-2.96" upper="2.96" velocity="0.5"/>

File: models/myArm_gripper.urdf (robot description, URDF)
Before this commit: robot Mitsubishi_rv-6sd, 9 links, 8 joints
Links:
- removed link body1
- removed link body10
- added link body20; visual cylinder length=0.8 radius=0.2
- added link body3; visual cylinder length=1 radius=0.2
Joints:
- removed joint j2
- removed joint j20
- added joint j30: type fixed, parent body2, child body20, origin xyz=0 0.2 0.7 rpy=0 0 0, axis 1 0 0, limit lower=-2.96 upper=2.96 effort=1000.0 velocity=0.5
- added joint j4: type revolute, parent body3, child gripper_pole, origin xyz=0 0 0.6 rpy=0 0 0, axis 0 1 0, limit lower=-2.96 upper=2.96 effort=1000.0 velocity=0.5
- joint base_joint: child body1 -> body2
- joint j3: child gripper_pole -> body3; origin xyz=0 0 0.6 rpy=0 0 0 -> xyz=0 0.2 0.3 rpy=0 0 0; parent body2 -> body20
