Commit message: Add Pisa hand joint information in C++

File: models/myArm_softHand.xacro (robot description, xacro)
@@ -212,5 +212,5 @@
 <joint name="j4" type="revolute">
     <parent link="body4"/>
-    <child link="softHandBase"/>
+    <child link="softHandWrist"/>
     <origin xyz="0 ${axel_offset} ${radius_hor_3+length4}" rpy="0 0 0"/>
     <axis xyz="0 0 1"/>
@@ -219,5 +219,5 @@
 </joint>
 <!---............................. HAND .............................................. -->
-<link name="softHandBase">
+<link name="softHandWrist">
     <collision> <!-- collision -->
         <origin rpy="0 0 0" xyz="0 0 ${length5/2}"/>
@@ -238,5 +238,5 @@
     </inertial>
 </link>
-<xacro:soft_hand name="softHand" parent="softHandBase"
+<xacro:soft_hand name="softHand" parent="softHandWrist"
                  withAdaptiveTransmission="true" useMimicTag="false" left="true">
   <origin xyz="0 0 ${length5/2}"

Commit message: Remove Kupa coupler, clamp and base, increase damping, decrease mass

File: models/myArm_softHand.xacro (robot description, xacro)
@@ -26,5 +26,5 @@
 <xacro:property name="length4"      value="${0.3 * scale}"   /> <!-- body 4 -->
 <xacro:property name="radius4"      value="${0.1 * scale}"   />
-<xacro:property name="length5"      value="${0.05 * scale}"  /> <!-- body 5 -->
+<xacro:property name="length5"      value="${0.03 * scale}"  /> <!-- body 5 -->
 <xacro:property name="radius5"      value="${0.05 * scale}"  />
 <xacro:property name="damping"      value="1" />             <!-- Damping -->
@@ -240,5 +240,5 @@
 <xacro:soft_hand name="softHand" parent="softHandWrist"
                  withAdaptiveTransmission="true" useMimicTag="false" left="true">
-  <origin xyz="0 0 ${length5/2}"
+  <origin xyz="0 0 0"
           rpy="0 0 0"/>
 </xacro:soft_hand>

File: models/pisa_iit_soft_hand/soft_hand.inertia.xacro (robot description, xacro)
@@ -10,5 +10,5 @@
     <xacro:property name="mm_to_m" value="0.001"/>
     <xacro:property name="mm2_to_m2" value="0.001"/>
-    <xacro:property name="gr_to_Kg" value="0.01"/>
+    <xacro:property name="gr_to_Kg" value="0.001"/>
     <!-- not so negligible, otherwise simulation fails -->
     <xacro:property name="negligible_mass" value="${10*gr_to_Kg}"/>

File: models/pisa_iit_soft_hand/soft_hand.urdf.xacro (robot description, xacro)
@@ -23,5 +23,5 @@
 	<xacro:property name="velocity" value="100" />
 	<xacro:property name="effort" value="100" />
-	<xacro:property name="damping" value="0.0" />
+    <xacro:property name="damping" value="10.0" />
 	<xacro:property name="friction" value="0.0" />
 	<!-- synergy vector -->
@@ -390,25 +390,13 @@
 	<xacro:macro name="soft_hand" params="parent name withAdaptiveTransmission useMimicTag left *origin">
 		<!-- PACMAN VERION ALREADY INCLUDES THE COUPLER, CLAMP AND BASE -->
-		<!-- KUKA_COUPLER -->
-		<xacro:kuka_coupler parent="${parent}" name="${name}_kuka_coupler">
-			<xacro:insert_block name="origin"/>
-		</xacro:kuka_coupler>
-		<!-- CLAMP -->
-		<xacro:clamp parent="${name}_kuka_coupler" name="${name}_clamp">
-			<origin xyz="0 0 0.01" rpy="0 0 0"/>
-		</xacro:clamp>
-		<!-- SOFT HAND BASE -->
-		<xacro:softhand_base parent="${name}_clamp" name="${name}_softhand_base" left="${left}">
-			<origin xyz="0 0 0.004" rpy="0 0 0"/>
-		</xacro:softhand_base>
 		<!-- PALM -->
 		<joint name="${name}_palm_joint" type="fixed">
 			<xacro:if value="${left}">
-				<origin xyz="0.002 -0.00695 0.0535" rpy="0 0 0"/>
+                <origin xyz="0 0 0" rpy="0 0 0"/>
 			</xacro:if>
 			<xacro:unless value="${left}">
-				<origin xyz="0.002 0.00695 0.0535" rpy="0 0 0"/>
+                <origin xyz="0 0 0" rpy="0 0 0"/>
 			</xacro:unless>
-			<parent link="${name}_softhand_base" />
+            <parent link="${parent}" />
 			<child link="${name}_palm_link" />
 		</joint>
